File: CM4.sch (EAGLE design)
At the start: 7 parts, among them J1 MAGJACK, J2 67800-5001, J3 RASPBERRYPI-40-PIN-GPIO_PTH_N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, J4 67800-5001, J5 67800-5001, J6 67800-5001

Commit message: finished board
Parts:
- removed J2: 67800-5001, SamacSys_Parts:67800-5001
- added BATT: (no value), SparkFun-Batteries:BATTERY-12MM_SMD
- added C1, C10, C11, C12, C13, C14, C15, C16, C17, C18, C19, C2, C22, C3, C32, C33, C34, C4, C5, C6, C7, C8, C9: 0.1uF, SparkFun-Capacitors:0.1UF-0603-25V-5%
- added C20: 1uF, SparkFun-Capacitors:0.1UF-0603-25V-5%
- added C21: 4.7uF, SparkFun-Capacitors:4.7UF-0603-6.3V-(10%)
- added C23: 10nF, SparkFun-Capacitors:4.7UF-0603-6.3V-(10%)
- added C24, C25: 18pF, SparkFun-Capacitors:0.1UF-0603-25V-5%
- added C26, C28, C30: 1uF, SparkFun-Capacitors:4.7UF-0603-6.3V-(10%)
- added C27, C29, C31: 2.2uF, SparkFun-Capacitors:4.7UF-0603-6.3V-(10%)
- added C35, C36, C37, C38: 865080640004, SamacSys_Parts:865080640004
- added D1: BAT54C, diode:BAT54C
- added IC1: PCF85063AT_AAZ, SamacSys_Parts:PCF85063AT_AAZ
- added IC2: MIC5504-1.8YM5-TR, SamacSys_Parts:MIC5504-1.8YM5-TR
- added IC3: REG1117, burr-brown:REG1117
- added IC4: W25X40CLSSIG, SamacSys_Parts:W25X40CLSSIG
- added IC5: ADP1740ACPZ-1.0-R7, SamacSys_Parts:ADP1740ACPZ-1.0-R7
- added J7: KUSBXHT-SLAS1N-O-HRF, SamacSys_Parts:KUSBXHT-SLAS1N-O-HRF
- added R1: 100k, rcl:R-US_R0603
- added R2: 6.04k, rcl:R-US_R0603
- added R3, R4: 10K, rcl:R-US_R0603
- added R5: 510k, rcl:R-US_R0603
- added R6: 510K, rcl:R-US_R0603
- added S1: MOMENTARY-SWITCH-SPST-SMD-5.2-REDUNDANT, SparkFun-Switches:MOMENTARY-SWITCH-SPST-SMD-5.2-REDUNDANT
- added U$2, U$3: SATA-D-PL-RT, SamacSys_Parts:SATA-D-PL-RT
- added U1: 88SE9215A1-NAA2C000, MarvellSATA:88SE9215A1-NAA2C000
- added U2: 74LVC1G07SE-7, SamacSys_Parts:74LVC1G07SE-7
- added X1: HDMI, raspberrypi_cm:HDMI
- added Y1: 25MHz, SparkFun-Clocks:CRYSTAL-25MHZ-SMD-2.0X1.6MM
- added Y2: 32.768kHz, SparkFun-Clocks:CRYSTAL-32.768KHZSMD-3.2X1.5
- J1: value MAGJACK -> (none); device SparkFun-Connectors:MAGJACK -> SparkFun-Connectors:CONN_06LOCK
- J3: value RASPBERRYPI-40-PIN-GPIO_PTH_NO_SHROUD -> COMPUTER_PERIPHERAL_POWERRA-VT; device SparkFun-Connectors:RASPBERRYPI-40-PIN-GPIO_PTH_NO_SHROUD -> SparkFun-Connectors:COMPUTER_PERIPHERAL_POWERRA-VT
- J4: value 67800-5001 -> 2250508-1; device SamacSys_Parts:67800-5001 -> SamacSys_Parts:2250508-1
- J5, J6: value 67800-5001 -> 8190-3; device SamacSys_Parts:67800-5001 -> SamacSys_Parts:8190-3
Connections:
- new net 1.0VDC: C21.1, C28.1, C29.1, IC5.SENSE, IC5.VOUT_1, IC5.VOUT_2, IC5.VOUT_3, IC5.VOUT_4, IC5.VOUT_5, U1.VDD, U1.VDD_2, U1.VDD_3, U1.VDD_4, U1.VDD_5, U1.VDD_6, U1.VDD_7
- new net 1.8VDC: C20.2, C26.1, C27.1, IC2.VOUT, U1.AVDD0, U1.VAA1, U1.VAA2_0, U1.VAA2_1, U1.VAA2_2, U1.VAA2_3
- new net 3V3: C22.2, C30.1, C31.1, C37.+, C38.+, D1.A2, IC3.VOUT, IC4.!HOLD, IC4.!WP, IC4.VCC, J1.4, U1.VDDIO, U1.VDDIO_2
- new net 5VDC: C34.2, C35.+, C36.+, IC2.EN, IC2.VIN, IC3.VIN, IC5.EN, IC5.VIN_1, IC5.VIN_2, IC5.VIN_3, IC5.VIN_4, IC5.VIN_5, J1.5, J3.5V, J7.1, R1.2, R5.2, R6.2, U$1POWER.5V-IN, U2.VCC, X1.+5V
- new net BUTTON: J1.6, U$1GPIO.GPIO15
- new net GLOBAL_EN: U$1SPECIAL-IO.GLOBAL_EN, U2.Y
- new net GND: BATT.-, C19.2, C20.1, C21.2, C22.1, C23.2, C24.1, C25.1, C26.2, C27.2, C28.2, C29.2, C30.2, C31.2, C33.2, C34.1, C35.-, C36.-, C37.-, C38.-, IC1.VSS, IC2.GND, IC3.GND, IC4.GND, IC5.EPAD, IC5.GND, J1.3, J3.GND@1, J3.GND@2, J7.4, R2.1, R3.1, R4.1, S1.2, U$1POWER.GND, U1.VSS, U1.VSS_2, U1.VSS_3, U1.VSS_4, U1.VSS_5, U2.GND, X1.GND@1, X1.GND@2, X1.GND@3, X1.GND@4, X1.GND@5, X1.GND@6, X1.GND@7, X1.GND@8, X1.GND@9
- new net HDMI_CK_N: U$1HDMI0.HDMI0_CK_N, X1.CLK_N
- new net HDMI_CK_P: U$1HDMI0.HDMI0_CK_P, X1.CLK_P
- new net HDMI_D0_N: U$1HDMI0.HDMI0_D0_N, X1.TX0_N
- new net HDMI_D0_P: U$1HDMI0.HDMI0_D0_P, X1.TX0_P
- new net HDMI_D1_N: U$1HDMI0.HDMI0_D1_N, X1.TX1_N
- new net HDMI_D1_P: U$1HDMI0.HDMI0_D1_P, X1.TX1_P
- new net HDMI_D2_N: U$1HDMI0.HDMI0_D2_N, X1.TX2_N
- new net HDMI_D2_P: U$1HDMI0.HDMI0_D2_P, X1.TX2_P
- new net N$1: C23.1, IC5.SS
- new net N$10: U$1HDMI0.HDMI0_SDA, X1.SDA
- new net N$11: U$1HDMI0.HDMI0_HOTPLUG, X1.HPD
- new net N$12: U$1HDMI0.HDMI0_CEC, X1.CEC_DAT
- new net N$13: IC1.OSCI, Y2.2
- new net N$14: IC1.OSCO, Y2.1
- new net N$16: C32.2, R6.1, U2.A
- new net N$18: J7.2, U$1USB.USB2_N
- new net N$19: J7.3, U$1USB.USB2_P
- new net N$24: BATT.+, D1.A1
- new net N$25: C19.1, D1.CC, IC1.VDD
- new net N$3: IC5.PG, R1.1
- new net N$4: C24.2, U1.XTLN_OSC, Y1.1
- new net N$5: C25.2, U1.XTLOUT, Y1.2
- new net N$6: C33.1, J4.TRCT1, J4.TRCT2, J4.TRCT3, J4.TRCT4
- new net N$67: R3.2, U1.TESTMODE
- new net N$68: U1.WAKE_N
- new net N$69: R4.2, U$1PCI-E.!PCIE_CLK_REQ
- new net N$7: S1.1, U$1SPECIAL-IO.!RPIBOOT
- new net N$8: R2.2, U1.ISET
- new net N$9: U$1HDMI0.HDMI0_SCL, X1.SCL
- new net NRTC_INT: C32.1, IC1.!INT, R5.1
- new net PCIERXCAP_N: C18.2, U$1PCI-E.PCIE_RX_N
- new net PCIERXCAP_P: C17.2, U$1PCI-E.PCIE_RX_P
- new net PCIERX_N: C18.1, U1.PTXP0
- new net PCIERX_P: C17.1, U1.PTXN0
- new net PCIETX_N: U$1PCI-E.PCIE_TX_N, U1.PRXP0
- new net PCIETX_P: U$1PCI-E.PCIE_TX_P, U1.PRXN0
- new net PCIE_CLK_N: U$1PCI-E.PCIE_CLK_P, U1.CLKP
- new net PCIE_CLK_P: U$1PCI-E.PCIE_CLK_N, U1.CLKN
- new net PCIE_RST: U$1PCI-E.!PCIE_RST, U1.PERST_N
- new net RX0_N: C14.2, U1.RXN_0
- new net RX0_P: C13.2, U1.RXP_0
- new net RX1_N: C10.2, U1.RXN_1
- new net RX1_P: C9.2, U1.RXP_1
- new net RX2_N: C6.2, U1.RXN_2
- new net RX2_P: C5.2, U1.RXP_2
- new net RX3_N: C2.2, U1.RXN_3
- new net RX3_P: C1.2, U1.RXP_3
- new net SATA1RX_N: C15.1, U$2.1_3
- new net SATA1RX_P: C16.1, U$2.1_2
- new net SATA1TX_N: C14.1, U$2.1_5
- new net SATA1TX_P: C13.1, U$2.1_6
- new net SATA1_GND: U$2.1_1, U$2.1_4, U$2.1_7
- new net SATA2RX_N: C11.1, U$2.2_3
- new net SATA2RX_P: C12.1, U$2.2_2
- new net SATA2TX_N: C10.1, U$2.2_5
- new net SATA2TX_P: C9.1, U$2.2_6
- new net SATA2_GND: U$2.2_1, U$2.2_4, U$2.2_7
- new net SATA3RX_N: C7.1, U$3.1_3
- new net SATA3RX_P: C8.1, U$3.1_2
- new net SATA3TX_N: C6.1, U$3.1_5
- new net SATA3TX_P: C5.1, U$3.1_6
- new net SATA3_GND: U$3.1_1, U$3.1_4, U$3.1_7
- new net SATA4RX_N: C3.1, U$3.2_3
- new net SATA4RX_P: C4.1, U$3.2_2
- new net SATA4TX_N: C2.1, U$3.2_5
- new net SATA4TX_P: C1.1, U$3.2_6
- new net SATA4_GND: U$3.2_1, U$3.2_4, U$3.2_7
- new net SCL: IC1.SCL, J1.2, U$1GPIO.SCL0
- new net SDA: IC1.SDA, J1.1, U$1GPIO.SDA0
- new net SPI_CLK: IC4.CLK, U1.SPI_CLK
- new net SPI_CS: IC4.!CS, U1.SPI_CS
- new net SPI_DI: IC4.DO(IO1), U1.SPI_DI
- new net SPI_DO: IC4.DI(IO0), U1.SPI_DO
- new net TRD0_N: J4.TRD1-, U$1ETHERNET.TRD0_N
- new net TRD0_P: J4.TRD1+, U$1ETHERNET.TRD0_P
- new net TRD1_N: J4.TRD2-, U$1ETHERNET.TRD1_N
- new net TRD1_P: J4.TRD2+, U$1ETHERNET.TRD1_P
- new net TRD2_N: J4.TRD3-, U$1ETHERNET.TRD2_N
- new net TRD2_P: J4.TRD3+, U$1ETHERNET.TRD2_P
- new net TRD3_N: J4.TRD4-, U$1ETHERNET.TRD3_N
- new net TRD3_P: J4.TRD4+, U$1ETHERNET.TRD3_P
- new net TX0_N: C15.2, U1.TXN_0
- new net TX0_P: C16.2, U1.TXP_0
- new net TX1_N: C11.2, U1.TXN_1
- new net TX1_P: C12.2, U1.TXP_1
- new net TX2_N: C7.2, U1.TXN_2
- new net TX2_P: C8.2, U1.TXP_2
- new net TX3_N: C3.2, U1.TXN_3
- new net TX3_P: C4.2, U1.TXP_3
Other:
- moved on the sheet: U$1ETHERNET, U$1GPIO, U$1PCI-E, U$1POWER, U$1USB
